File: kicad-files/dc_programmable_load/dc_programmable_load.kicad_pcb (KiCad board)
At the start: 2 copper layers, 49 x 58.5 mm, 38 parts, among them J1 DC Jack 12V, J10 Conn_01x01_Socket, J11 Conn_01x01_Socket, J12 Conn_01x01_Socket, J13 Conn_01x01_Socket, J14 Conn_01x01_Socket, J2 Conn_01x03_Socket, J5 Conn_01x01_Socket, J6 Conn_01x01_Socket, J7 Conn_01x03_Socket, J8 Conn_01x03_Socket, J9 Conn_01x01_Socket, Q1 IRF3205, U1 LM358DR, U3 AP63200WU

Commit message: Update KiCad PCB, schematic, and project layout files
Co-Authored-By: Claude Opus 4.8 (1M context) <noreply@anthropic.com>
Parts:
- renumbered TempSnsr1 to TS1
Routing:
- net GND: vias 121 -> 127
Changed lines of the file:
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@@
 		(tags "SOT TO_SOT_SMD")
 		(property "Reference" "DAC1"
-			(at 0 -2.4 90)
+			(at -0.6375 -3.45 90)
 			(layer "F.SilkS")
 			(effects
@@
 		(tags "SRR4028-4R7Y ")
 		(property "Reference" "L1"
-			(at 0 0 0)
+			(at 0 4 0)
 			(unlocked yes)
 			(layer "F.SilkS")
@@
 			(layer "F.SilkS")
 		)
-		(fp_line
-			(start -3.0099 -2.9083)
-			(end -2.7559 -2.9083)
-			(stroke
-				(width 0.1524)
-				(type solid)
-			)
-			(layer "F.CrtYd")
-		)
-		(fp_line
-			(start -3.0099 2.9083)
-			(end -3.0099 -2.9083)
-			(stroke
-				(width 0.1524)
-				(type solid)
-			)
-			(layer "F.CrtYd")
-		)
-		(fp_line
-			(start -2.7559 -2.9083)
-			(end -2.7559 -2.9083)
-			(stroke
-				(width 0.1524)
-				(type solid)
-			)
-			(layer "F.CrtYd")
-		)
-		(fp_line
-			(start -2.7559 -2.9083)
-			(end 2.7559 -2.9083)
-			(stroke
-				(width 0.1524)
-				(type solid)
-			)
-			(layer "F.CrtYd")
-		)
-		(fp_line
-			(start -2.7559 2.9083)
-			(end -3.0099 2.9083)
-			(stroke
-				(width 0.1524)
-				(type solid)
-			)
-			(layer "F.CrtYd")
-		)
-		(fp_line
-			(start -2.7559 2.9083)
-			(end -2.7559 2.9083)
-			(stroke
-				(width 0.1524)
-				(type solid)
-			)
-			(layer "F.CrtYd")
-		)
-		(fp_line
-			(start 2.7559 -2.9083)
-			(end 2.7559 -2.9083)
-			(stroke
-				(width 0.1524)
-				(type solid)
-			)
-			(layer "F.CrtYd")
-		)
-		(fp_line
-			(start 2.7559 -2.9083)
-			(end 3.0099 -2.9083)
-			(stroke
-				(width 0.1524)
-				(type solid)
-			)
-			(layer "F.CrtYd")
-		)
-		(fp_line
-			(start 2.7559 2.9083)
-			(end -2.7559 2.9083)
-			(stroke
-				(width 0.1524)
-				(type solid)
-			)
-			(layer "F.CrtYd")
-		)
-		(fp_line
-			(start 2.7559 2.9083)
-			(end 2.7559 2.9083)
-			(stroke
-				(width 0.1524)
-				(type solid)
-			)
-			(layer "F.CrtYd")
-		)
-		(fp_line
-			(start 3.0099 -2.9083)
-			(end 3.0099 2.9083)
-			(stroke
-				(width 0.1524)
-				(type solid)
-			)
-			(layer "F.CrtYd")
-		)
-		(fp_line
-			(start 3.0099 2.9083)
-			(end 2.7559 2.9083)
+		(fp_rect
+			(start -3 -3)
+			(end 3 3)
 			(stroke
-				(width 0.1524)
-				(type solid)
+				(width 0.05)
+				(type default)
 			)
+			(fill no)
 			(layer "F.CrtYd")
 		)
@@
 		)
 		(fp_text user "${REFERENCE}"
-			(at 0 0 0)
+			(at 0 4 0)
 			(unlocked yes)
 			(layer "F.Fab")
@@
 		(descr "DFN, 8 Pin (http://ww1.microchip.com/downloads/en/DeviceDoc/8L_DFN_2x3x0_9_MC_C04-123C.pdf)")
 		(tags "DFN NoLead")
-		(property "Reference" "TempSnsr1"
-			(at 0 -1.95 0)
+		(property "Reference" "TS1"
+			(at -0.075 1.85 0)
 			(layer "F.SilkS")
 			(effects
@@
 			(layers "F.Cu" "F.Mask" "F.Paste")
 			(roundrect_rratio 0.25)
-			(net "unconnected-(TempSnsr1-Alert-Pad3)")
+			(net "unconnected-(TS1-Alert-Pad3)")
 			(pinfunction "Alert_3")
 			(pintype "output+no_connect")
@@
 		(tags "capacitor")
 		(property "Reference" "C7"
-			(at -1 -1.5 90)
+			(at -1.5 -1.5 90)
 			(layer "F.SilkS")
 			(effects
@@
 		(tags "Through hole pin header THT 1x01 2.00mm single row")
 		(property "Reference" "J12"
-			(at 0 -2.11 0)
+			(at -1 -2.11 0)
 			(layer "F.SilkS")
 			(effects
@@
 		(tags "capacitor")
 		(property "Reference" "C8"
-			(at 0 -1.68 90)
+			(at 0.5 2 90)
 			(layer "F.SilkS")
 			(effects
@@
 	)
 	(via
-		(at 170.460456 95.033867)
+		(at 170.5 97)
 		(size 0.6)
 		(drill 0.3)
@@
 	)
 	(via
+		(at 138.5 94.5)
+		(size 0.6)
+		(drill 0.3)
+		(layers "F.Cu" "B.Cu")
+		(free yes)
+		(net "GND")
+	)
+	(via
 		(at 156 61.700682)
 		(size 0.6)
@@
 	)
 	(via
+		(at 134.5 97)
+		(size 0.6)
+		(drill 0.3)
+		(layers "F.Cu" "B.Cu")
+		(free yes)
+		(net "GND")
+	)
+	(via
 		(at 130 72)
 		(size 0.6)
@@
 	)
 	(via
-		(at 170.5 90)
+		(at 170 91)
 		(size 0.6)
 		(drill 0.3)
@@
 	)
 	(via
-		(at 135.632946 97.532416)
+		(at 136 97.5)
 		(size 0.6)
 		(drill 0.3)
@@
 	)
 	(via
+		(at 136.5 94)
+		(size 0.6)
+		(drill 0.3)
+		(layers "F.Cu" "B.Cu")
+		(free yes)
+		(net "GND")
+	)
+	(via
 		(at 165 81)
 		(size 0.6)
@@
 	)
 	(via
+		(at 144 95.5)
+		(size 0.6)
+		(drill 0.3)
+		(layers "F.Cu" "B.Cu")
+		(free yes)
+		(net "GND")
+	)
+	(via
+		(at 140 93.5)
+		(size 0.6)
+		(drill 0.3)
+		(layers "F.Cu" "B.Cu")
+		(free yes)
+		(net "GND")
+	)
+	(via
 		(at 141.890889 87.192184)
 		(size 0.6)
@@
 		(size 0.6)
 		(drill 0.3)
+		(layers "F.Cu" "B.Cu")
+		(free yes)
+		(net "GND")
+	)
+	(via
+		(at 171 93.5)
+		(size 0.6)
+		(drill 0.3)
