File: kicad-files/dc_programmable_load/dc_programmable_load.kicad_pcb (KiCad board)
At the start: 2 copper layers, 49 x 58.5 mm, 38 parts, among them J1 DC Jack 12V, J10 Conn_01x01_Socket, J11 Conn_01x01_Socket, J12 Conn_01x01_Socket, J13 Conn_01x01_Socket, J14 Conn_01x01_Socket, J2 Conn_01x03_Socket, J5 Conn_01x01_Socket, J6 Conn_01x01_Socket, J7 Conn_01x03_Socket, J8 Conn_01x03_Socket, J9 Conn_01x01_Socket, Q1 IRF3205, U1 LM358DR, U3 AP63200WU

Commit message: should be final version
Parts:
- moved R1 0.50 mm to (126.0, 75.0)
Routing:
- net GND: vias 127 -> 129
Other:
- board size 49 x 58.5 mm -> 49 x 59 mm
Changed lines of the file:
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@@
 	(footprint "Resistor_SMD:R_0805_2012Metric"
 		(layer "F.Cu")
-		(at 125.5 75 -90)
+		(at 126 75 -90)
 		(descr "Resistor SMD 0805 (2012 Metric), square (rectangular) end terminal, IPC-7351 nominal, (Body size source: IPC-SM-782 page 72, https://www.pcb-3d.com/wordpress/wp-content/uploads/ipc-sm-782a_amendment_1_and_2.pdf)")
 		(tags "resistor")
@@
 	)
 	(gr_rect
-		(start 124 60.5)
+		(start 124 60)
 		(end 173 119)
 		(stroke
@@
 	)
 	(segment
-		(start 128.5 83)
-		(end 128.5 82.5)
+		(start 132.5 85)
+		(end 135 87.5)
 		(width 1)
 		(layer "F.Cu")
@@
 	)
 	(segment
-		(start 132.5 85)
-		(end 135 87.5)
+		(start 128.5 83)
+		(end 128.5 83.65)
 		(width 1)
 		(layer "F.Cu")
@@
 	(segment
 		(start 128.5 83)
-		(end 128.5 83.65)
+		(end 128.5 82.5)
+		(width 1)
+		(layer "F.Cu")
+		(net "/A2")
+	)
+	(segment
+		(start 128.5 82.5)
+		(end 126 80)
 		(width 1)
 		(layer "F.Cu")
@@
 	)
 	(segment
-		(start 125.5 79.5)
-		(end 125.5 75.9125)
-		(width 1)
-		(layer "F.Cu")
-		(net "/A2")
-	)
-	(segment
-		(start 128.5 82.5)
-		(end 125.5 79.5)
+		(start 126 80)
+		(end 126 75.9125)
 		(width 1)
 		(layer "F.Cu")
@@
 	)
 	(via
+		(at 137.5 61)
+		(size 0.6)
+		(drill 0.3)
+		(layers "F.Cu" "B.Cu")
+		(free yes)
+		(net "GND")
+	)
+	(via
 		(at 146 71.5)
 		(size 0.6)
@@
 	)
 	(via
-		(at 125.04 63.05)
+		(at 125.5 63.5)
 		(size 0.6)
 		(drill 0.3)
@@
 	)
 	(via
-		(at 127.04 62.55)
+		(at 127.5 61.5)
 		(size 0.6)
 		(drill 0.3)
@@
 	)
 	(via
-		(at 172 62.200682)
+		(at 171.5 62.5)
 		(size 0.6)
 		(drill 0.3)
@@
 	)
 	(via
+		(at 131.5 61)
+		(size 0.6)
+		(drill 0.3)
+		(layers "F.Cu" "B.Cu")
+		(free yes)
+		(net "GND")
+	)
+	(via
 		(at 138.714716 83.674487)
 		(size 0.6)
@@
 	)
 	(segment
-		(start 136.54 62.55)
-		(end 130.04 62.55)
-		(width 1)
-		(layer "F.Cu")
-		(net "/Power Supply")
-	)
-	(segment
 		(start 144 72.725)
 		(end 145.225 72.725)
@@
 	)
 	(segment
-		(start 125.5 67)
-		(end 125.5 74.0875)
-		(width 1)
-		(layer "F.Cu")
-		(net "/Power Supply")
-	)
-	(segment
 		(start 145.225 72.725)
 		(end 142.04 69.54)
@@
 	)
 	(segment
-		(start 130.04 62.55)
-		(end 125.54 67.05)
-		(width 1)
-		(layer "F.Cu")
-		(net "/Power Supply")
-	)
-	(segment
 		(start 153.5 79.5)
 		(end 153.5 79)
@@
 	)
 	(segment
+		(start 136.54 62.55)
+		(end 129.95 62.55)
+		(width 1)
+		(layer "F.Cu")
+		(net "/Power Supply")
+	)
+	(segment
 		(start 155.2474 79.5)
 		(end 153.5 79.5)
@@
 	)
 	(segment
+		(start 126 66.5)
+		(end 126 74.0875)
+		(width 1)
+		(layer "F.Cu")
+		(net "/Power Supply")
+	)
+	(segment
 		(start 153.5 79.5)
 		(end 152 79.5)
@@
 	)
 	(segment
+		(start 129.95 62.55)
+		(end 126 66.5)
+		(width 1)
+		(layer "F.Cu")
+		(net "/Power Supply")
+	)
+	(segment
 		(start 141 91)
 		(end 142 90)
@@
 		(polygon
 			(pts
-				(xy 124.5 61) (xy 172.5 61) (xy 172.5 104) (xy 124.5 104)
+				(xy 124.5 60.5) (xy 172.5 60.5) (xy 172.5 104) (xy 124.5 104)
 			)
 		)
