File: kicad-files/dc_programmable_load/dc_programmable_load.kicad_pcb (KiCad board)
At the start: 2 copper layers, 49 x 59 mm, 38 parts, among them J1 DC Jack 12V, J10 Conn_01x01_Socket, J11 Conn_01x01_Socket, J12 Conn_01x01_Socket, J13 Conn_01x01_Socket, J14 Conn_01x01_Socket, J2 Conn_01x03_Socket, J5 Conn_01x01_Socket, J6 Conn_01x01_Socket, J7 Conn_01x03_Socket, J8 Conn_01x03_Socket, J9 Conn_01x01_Socket, Q1 IRF3205, U1 LM358DR, U3 AP63200WU

Commit message: Add v2 and m1_key KiCad designs; ignore .history dumps
Co-Authored-By: Claude Opus 4.8 (1M context) <noreply@anthropic.com>
Parts:
- added U2: ER_OLEDM0.91_1x-I2C, Display:ER_OLEDM0.91_1x-I2C, F.Cu at (184.5, 98.0)
