File: kicad-files/dc_programmable_load_m1_key/dc_programmable_load_m1_key.kicad_pcb (KiCad board)
At the start: 2 copper layers, 65 x 65 mm, 26 parts, among them J1 DC Jack 12V, Q1 IRF3205, U1 LM358DR, U2 ER_OLEDM0.91_1x-I2C

Commit message: Update v2 design files and m1_key PCB
Co-Authored-By: Claude Opus 4.8 (1M context) <noreply@anthropic.com>
Changed lines of the file:
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@@
 	)
 	(segment
-		(start 131.5 79)
-		(end 136 79)
-		(width 1)
-		(layer "F.Cu")
-		(net "/opamp_output")
-	)
-	(segment
-		(start 141 74)
-		(end 141 71.0875)
+		(start 128 75.5)
+		(end 131.5 79)
 		(width 1)
 		(layer "F.Cu")
@@
 	)
 	(segment
-		(start 141 71.0875)
-		(end 141.5875 70.5)
+		(start 141.5 73.5)
+		(end 141.5 70.5875)
 		(width 1)
 		(layer "F.Cu")
@@
 		(start 128 75.5)
 		(end 131.0875 75.5)
+		(width 1)
+		(layer "F.Cu")
+		(net "/opamp_output")
+	)
+	(segment
+		(start 131.5 79)
+		(end 136 79)
 		(width 1)
 		(layer "F.Cu")
@@
 	(segment
 		(start 136 79)
-		(end 141 74)
+		(end 141.5 73.5)
 		(width 1)
 		(layer "F.Cu")
@@
 	)
 	(segment
-		(start 128 75.5)
-		(end 131.5 79)
+		(start 141.5 70.5875)
+		(end 141.5875 70.5)
 		(width 1)
 		(layer "F.Cu")
