File: kicad-files/dc_programmable_load_v2/dc_programmable_load_v2.kicad_pcb (KiCad board)
At the start: 2 copper layers, 80 x 80 mm, 42 parts, among them J1 DC Jack 12V, J2 Conn_01x03_Socket, J3 Conn_01x04_Socket, Q1 IRF3205, U1 LM358DR, U2 ER_OLEDM0.91_1x-I2C, U3 AP63200WU, U5 S-2050

Commit message: Update v2 PCB, schematic, and project files
Co-Authored-By: Claude Opus 4.8 (1M context) <noreply@anthropic.com>
Parts:
- removed J2: Conn_01x03_Socket, Connector_PinHeader_2.00mm:PinHeader_1x03_P2.00mm_Vertical
- removed TS1: MCP9808_DFN, Package_DFN_QFN:DFN-8-1EP_3x2mm_P0.5mm_EP1.7x1.4mm
- added F1: Fuse, Fuse:Fuse_1210_3225Metric, F.Cu at (159.5, 74.0)
- added R4: 4.7k, Resistor_SMD:R_0805_2012Metric, F.Cu at (136.5, 62.5)
- added U4: DS18B20, Package_TO_SOT_THT:TO-92_Inline, F.Cu at (147.0, 64.0)
- moved C14 13.3 mm to (169.5, 79.2)
- moved C15 13.1 mm to (173.0, 79.2)
- moved Shunt1 11.3 mm to (151.5, 88.2)
- moved C10 6.17 mm to (142.2, 62.2), turned to -90 degrees
- moved R1 6.07 mm to (142.0, 81.3)
- moved R6 3.27 mm to (152.5, 76.2)
- moved Q1 3.27 mm to (150.6, 69.3)
- moved R2 0.90 mm to (141.0, 87.8)
Connections:
- A1 pad 20: unconnected-(A1-A1-Pad20) -> /temp_pin1
- C14 pad 2: /Power Supply -> /nettop1
- C15 pad 2: /Power Supply -> /nettop1
- L1 pad 1: /Power Supply -> /nettop1
- R10 pad 1: /Power Supply -> /nettop1
- R11 pad 1: /Power Supply -> /nettop1
- R12 pad 1: /Power Supply -> /nettop1
- R9 pad 1: /Power Supply -> /nettop1
Routing:
- net /temp_pin1: track 0.00 -> 139.2 mm
- net /sda: track 166.4 -> 49.6 mm
- net /scl: track 156.1 -> 47.2 mm
- net /Power Supply: track 88.6 -> 36.6 mm
- net /nettop1: track 0.00 -> 44.1 mm
- net /3v3: track 157.3 -> 169.9 mm
- net Net-(J2-Pin_3): track 8.54 -> 0.00 mm
- net Net-(J2-Pin_2): track 8.45 -> 0.00 mm
- net /A2: track 39.3 -> 31.0 mm
- net Net-(J2-Pin_1): track 7.95 -> 0.00 mm
- net /A0: track 48.0 -> 46.4 mm
- net /opamp_output: track 45.6 -> 44.2 mm
- net GND: vias 240 -> 255
Other:
- board text added: "Short Circuit DC Programmable Load"

Commit message: Update v2 design files and m1_key PCB
Co-Authored-By: Claude Opus 4.8 (1M context) <noreply@anthropic.com>
Parts:
- 3v3, GND1: value Conn_01x03_Socket -> Conn_01x02_Socket; footprint Connector_PinHeader_2.00mm:PinHeader_1x03_P2.00mm_Vertical -> Connector_PinHeader_2.54mm:PinHeader_1x02_P2.54mm_Vertical
- J3: footprint Connector_PinHeader_2.00mm:PinHeader_1x04_P2.00mm_Vertical -> Connector_PinHeader_2.54mm:PinHeader_1x04_P2.54mm_Vertical
- Res1, Res2, SDA/SCL1: footprint Connector_PinHeader_2.00mm:PinHeader_1x02_P2.00mm_Vertical -> Connector_PinHeader_2.54mm:PinHeader_1x02_P2.54mm_Vertical
- moved GND1 8.76 mm to (194.2, 112.5), turned to -90 degrees
- moved C10 4.27 mm to (138.0, 62.2)
- moved R4 4.27 mm to (132.2, 62.5)
- moved U4 4.27 mm to (142.7, 64.0)
- moved Q1 4.27 mm to (146.3, 69.3)
- moved 3v3 4.26 mm to (189.8, 118.2), turned to -90 degrees
- moved R1 2.50 mm to (139.5, 81.2)
- moved R6 2.27 mm to (150.5, 75.2), turned to 180 degrees
- moved Res2 1.75 mm to (160.5, 102.8)
- moved J3 0.79 mm to (134.3, 137.5)
Routing:
- net /3v3: track 169.9 -> 163.9 mm
- net /temp_pin1: track 139.2 -> 134.9 mm
- net /A0: track 46.4 -> 49.0 mm
- net /opamp_output: track 44.2 -> 46.8 mm
- net /Power Supply: track 36.6 -> 39.1 mm
- net Net-(Q1-G): track 7.38 -> 8.67 mm
- net /A2: track 31.0 -> 32.2 mm
- net Net-(Res1-Pin_1): track 40.1 -> 40.8 mm
