File: kicad-files/dc_programmable_load_v2/dc_programmable_load_v2.kicad_pcb (KiCad board)
At the start: 2 copper layers, 80 x 80 mm, 43 parts, among them J1 DC Jack 12V, J3 Conn_01x04_Socket, Q1 IRF3205, U1 LM358DR, U2 ER_OLEDM0.91_1x-I2C, U3 AP63200WU, U4 DS18B20, U5 S-2050

Commit message: anand newest edits
Parts:
- removed U5: S-2050, s-2050:S-2050_NDC
- added S1: PEC11R-4015F-S0024, pec:XDCR_PEC11R-4015F-S0024, F.Cu at (198.5, 83.5)
- moved R12 29.6 mm to (209.1, 86.0), turned to 180 degrees
- moved R11 29.5 mm to (209.1, 81.0), turned to 180 degrees
- moved L1 15.3 mm to (201.7, 97.0), turned to 180 degrees
- moved R9 6.57 mm to (184.5, 81.0)
- moved R10 5.83 mm to (184.5, 86.0), turned to 180 degrees
- moved C14 5.00 mm to (174.5, 79.3)
- moved C15 5.00 mm to (178.0, 79.3)
Connections:
- R10 pad 1: /nettop1 -> Net-(R10-Pad1)
- R10 pad 2: Net-(R10-Pad2) -> /nettop1
Routing:
- net /12V: track 85.7 -> 119.8 mm
- net /nettop1: track 44.1 -> 76.4 mm, vias 0 -> 2
- net Net-(U3-SW): track 51.7 -> 58.6 mm
- net Net-(R10-Pad1): track 0.00 -> 5.59 mm
- net Net-(R10-Pad2): track 5.37 -> 0.00 mm
- net /netbot1: track 29.4 -> 31.3 mm
- net Net-(R12-Pad2): track 4.36 -> 2.68 mm
- net Net-(R11-Pad2): track 4.03 -> 2.68 mm
- net Net-(R9-Pad2): track 4.75 -> 5.59 mm
- net GND: vias 255 -> 247
Other:
- board size 80 x 80 mm -> 95 x 79.5 mm
