File: kicad-files/dc_programmable_load_v2/dc_programmable_load_v2.kicad_sch (KiCad schematic)
At the start: 42 parts, among them J1 DC Jack 12V, J2 Conn_01x03_Socket, J3 Conn_01x04_Socket, Q1 IRF3205, U1 LM358DR, U2 ER_OLEDM0.91_1x-I2C, U3 AP63200WU, U5 S-2050

Commit message: Update v2 PCB, schematic, and project files
Co-Authored-By: Claude Opus 4.8 (1M context) <noreply@anthropic.com>
Parts:
- removed J2: Conn_01x03_Socket, Connector_PinHeader_2.00mm:PinHeader_1x03_P2.00mm_Vertical, symbol Connector:Conn_01x03_Socket
- removed TS1: MCP9808_DFN, Package_DFN_QFN:DFN-8-1EP_3x2mm_P0.5mm_EP1.7x1.4mm, symbol Sensor_Temperature:MCP9808_DFN
- added F1: Fuse, Fuse:Fuse_1210_3225Metric, symbol Device:Fuse
- added R4: 4.7k, Resistor_SMD:R_0805_2012Metric, symbol Device:R
- added U4: DS18B20, Package_TO_SOT_THT:TO-92_Inline, symbol Sensor_Temperature:DS18B20
Connections:
- net 3v3: now also R4.1, U4.3 (V_{DD})
- net GND: now also U4.1 (GND)
- net Power Supply: now also F1.2; no longer C14.2, C15.2, L1.1, R10.1, R11.1, R12.1, R9.1
- net temp_pin1: now reaches A1.20 (A1)
- net temp_pin1: now also R4.2, U4.2 (DQ)
- new net nettop1: C14.2, C15.2, F1.1, L1.1, R10.1, R11.1, R12.1, R9.1
- no-connect marks 30 -> 28
Other:
- moved on the sheet: C10

Commit message: Update v2 design files and m1_key PCB
Co-Authored-By: Claude Opus 4.8 (1M context) <noreply@anthropic.com>
Parts:
- removed 3v3, GND1: Conn_01x03_Socket, Connector_PinHeader_2.00mm:PinHeader_1x03_P2.00mm_Vertical, symbol Connector:Conn_01x03_Socket
- added 3v3, GND1: Conn_01x02_Socket, Connector_PinHeader_2.54mm:PinHeader_1x02_P2.54mm_Vertical, symbol Connector:Conn_01x02_Socket
- J3: footprint Connector_PinHeader_2.00mm:PinHeader_1x04_P2.00mm_Vertical -> Connector_PinHeader_2.54mm:PinHeader_1x04_P2.54mm_Vertical
- Res1, Res2, SDA/SCL1: footprint Connector_PinHeader_2.00mm:PinHeader_1x02_P2.00mm_Vertical -> Connector_PinHeader_2.54mm:PinHeader_1x02_P2.54mm_Vertical
Connections:
- net 3v3: now also 3v3.1 (Pin_1), 3v3.2 (Pin_2)
- net GND: now also GND1.1 (Pin_1), GND1.2 (Pin_2)
